Commit message: Refresh K1 assets: height 1355 mm, render/imitation images, and latest URDF meshes.
Co-authored-by: Cursor <cursoragent@cursor.com>

File: docusaurus/static/assets/aisapiens/k1/ai_sapiens_description/urdf/k1_rev1/k1_rev1.urdf.xacro (robot description, xacro)
@@ -1,8 +1,5 @@
 <?xml version="1.0" ?>
-<!-- =================================================================================== -->
-<!-- | This document was autogenerated by xacro from /root/ros2_ws/src/ai_sapiens/ai_sapiens_description/urdf/k1_rev1/k1.urdf.xacro | -->
-<!-- |    EDITING THIS FILE BY HAND IS NOT RECOMMENDED                                 | -->
-<!-- =================================================================================== -->
-<robot name="k1">
+<robot xmlns:xacro="http://www.ros.org/wiki/xacro">
+<xacro:macro name="k1">
   <material name="dark">
     <color rgba="0.2 0.2 0.2 1"/>
@@ -32,7 +29,9 @@
     </collision>
     <inertial>
-      <origin xyz="6.953003800e-03 3.242849800e-06 1.065532100e-01"/>
-      <mass value="7.279675100e-01"/>
-      <inertia ixx="2.638882900e-03" ixy="-1.118249400e-07" ixz="2.006416200e-04" iyy="2.937964300e-03" iyz="-3.616676400e-08" izz="1.817875800e-03"/>
+      <origin xyz="6.953003800e-03 3.242849800e-06 1.065532100e-01" />
+      <mass value="7.279675100e-01" />
+      <inertia ixx="2.638882900e-03" ixy="-1.118249400e-07" ixz="2.006416200e-04"
+                iyy="2.937964300e-03" iyz="-3.616676400e-08"
+                izz="1.817875800e-03" />
     </inertial>
   </link>
@@ -52,7 +51,9 @@
     </collision> -->
     <inertial>
-      <origin xyz="-2.926489100e-03 1.127755300e-06 -5.031535600e-02"/>
-      <mass value="3.611882200e+00"/>
-      <inertia ixx="1.310639100e-02" ixy="-2.328809400e-07" ixz="5.514559000e-05" iyy="9.174952600e-03" iyz="0.000000000e+00" izz="7.736608000e-03"/>
+       <origin xyz="-2.926489100e-03 1.127755300e-06 -5.031535600e-02" />
+       <mass value="3.611882200e+00" />
+       <inertia ixx="1.310639100e-02" ixy="-2.328809400e-07" ixz="5.514559000e-05"
+       iyy="9.174952600e-03" iyz="0.000000000e+00"
+       izz="7.736608000e-03" />
     </inertial>
   </link>
@@ -67,13 +68,15 @@
     </visual>
     <collision>
-      <origin rpy="1.5708 0 0" xyz="0 0.05 -0.02"/>
-      <geometry>
-        <cylinder length="0.07" radius="0.04"/>
-      </geometry>
-    </collision>
-    <inertial>
-      <origin xyz="-1.141670400e-03 7.948432600e-02 -2.579805100e-02"/>
-      <mass value="1.134347800e+00"/>
-      <inertia ixx="1.413286200e-03" ixy="1.518924500e-05" ixz="-1.201272000e-05" iyy="1.011148100e-03" iyz="1.525829600e-04" izz="1.066244600e-03"/>
+      <origin xyz="0 0.05 -0.02" rpy="1.5708 0 0"/>
+      <geometry>
+        <cylinder radius="0.04" length="0.07"/>
+      </geometry>
+    </collision>
+    <inertial>
+       <origin xyz="-1.141670400e-03 7.948432600e-02 -2.579805100e-02" />
+       <mass value="1.134347800e+00" />
+       <inertia ixx="1.413286200e-03" ixy="1.518924500e-05" ixz="-1.201272000e-05"
+       iyy="1.011148100e-03" iyz="1.525829600e-04"
+       izz="1.066244600e-03" />
     </inertial>
   </link>
@@ -94,7 +97,9 @@
     </visual>
     <inertial>
-      <origin xyz="1.451722900e-02 -2.959881100e-06 -7.908222600e-02"/>
-      <mass value="1.553530600e+00"/>
-      <inertia ixx="2.895595600e-03" ixy="2.404258600e-07" ixz="-7.419442800e-05" iyy="3.373316500e-03" iyz="-2.099420700e-07" izz="1.930198000e-03"/>
+       <origin xyz="1.451722900e-02 -2.959881100e-06 -7.908222600e-02" />
+       <mass value="1.553530600e+00" />
+       <inertia ixx="2.895595600e-03" ixy="2.404258600e-07" ixz="-7.419442800e-05"
+       iyy="3.373316500e-03" iyz="-2.099420700e-07"
+       izz="1.930198000e-03" />
     </inertial>
   </link>
@@ -115,13 +120,15 @@
     </visual>
     <collision>
-      <origin rpy="0 0 0" xyz="0.0 0 -0.08"/>
-      <geometry>
-        <cylinder length="0.13" radius="0.045"/>
-      </geometry>
-    </collision>
-    <inertial>
-      <origin xyz="-1.981771700e-03 -4.936338800e-03 -1.811417900e-01"/>
-      <mass value="1.898213600e+00"/>
-      <inertia ixx="1.106385300e-02" ixy="-5.976117400e-05" ixz="-4.863131900e-04" iyy="1.147674900e-02" iyz="-6.115589000e-04" izz="1.632573000e-03"/>
+      <origin xyz="0.0 0 -0.08" rpy="0 0 0"/>
+      <geometry>
+        <cylinder radius="0.045" length="0.13"/>
+      </geometry>
+    </collision>
+    <inertial>
+       <origin xyz="-1.981771700e-03 -4.936338800e-03 -1.811417900e-01" />
+       <mass value="1.898213600e+00" />
+       <inertia ixx="1.106385300e-02" ixy="-5.976117400e-05" ixz="-4.863131900e-04"
+       iyy="1.147674900e-02" iyz="-6.115589000e-04"
+       izz="1.632573000e-03" />
     </inertial>
   </link>
@@ -141,13 +148,15 @@
       <material name="white"/>
     </visual>
-    <inertial>
-      <origin xyz="-3.870294200e-04 3.148109200e-03 -1.238798000e-01"/>
-      <mass value="2.340311200e+00"/>
-      <inertia ixx="1.081088800e-02" ixy="1.641625300e-04" ixz="-2.747466700e-04" iyy="1.105245000e-02" iyz="-3.835456300e-04" izz="2.561741000e-03"/>
-    </inertial>
-    <collision>
-      <origin rpy="0 0 0" xyz="0.0 0 -0.10"/>
-      <geometry>
-        <cylinder length="0.18" radius="0.04"/>
+     <inertial>
+        <origin xyz="-3.870294200e-04 3.148109200e-03 -1.238798000e-01" />
+        <mass value="2.340311200e+00" />
+        <inertia ixx="1.081088800e-02" ixy="1.641625300e-04" ixz="-2.747466700e-04"
+        iyy="1.105245000e-02" iyz="-3.835456300e-04"
+        izz="2.561741000e-03" />
+     </inertial>
+    <collision>
+      <origin xyz="0.0 0 -0.10" rpy="0 0 0"/>
+      <geometry>
+        <cylinder radius="0.04" length="0.18"/>
       </geometry>
     </collision>
@@ -175,7 +184,9 @@
     </collision>-->
     <inertial>
-      <origin xyz="5.032473200e-03 -3.766079000e-05 2.402319500e-03"/>
-      <mass value="6.779372600e-01"/>
-      <inertia ixx="3.704684500e-04" ixy="-1.179149700e-06" ixz="4.766622000e-05" iyy="4.135993600e-04" iyz="5.727227700e-07" izz="4.302869000e-04"/>
+      <origin xyz="5.032473200e-03 -3.766079000e-05 2.402319500e-03" />
+      <mass value="6.779372600e-01" />
+      <inertia ixx="3.704684500e-04" ixy="-1.179149700e-06" ixz="4.766622000e-05"
+                iyy="4.135993600e-04" iyz="5.727227700e-07"
+                izz="4.302869000e-04" />
     </inertial>
   </link>
@@ -195,68 +206,16 @@
       <material name="white"/>
     </visual>
-    <!-- <collision>
+    <collision>
       <origin rpy="0 0 0" xyz="0 0 0"/>
       <geometry>
         <mesh filename="package://ai_sapiens_description/meshes/k1_rev1/left_ankle_roll_link.stl" scale="0.001 0.001 0.001"/>
       </geometry>
-    </collision> -->
-    <collision>
-      <origin rpy="0 0 0" xyz="-0.047 0.025 -0.06"/>
-      <geometry>
-        <sphere radius="0.005"/>
-      </geometry>
-    </collision>
-    <collision>
-      <origin rpy="0 0 0" xyz="-0.047 -0.025 -0.06"/>
-      <geometry>
-        <sphere radius="0.005"/>
-      </geometry>
-    </collision>
-    <collision>
-      <origin rpy="0 0 0" xyz="0.05 0.038 -0.06"/>
-      <geometry>
-        <sphere radius="0.005"/>
-      </geometry>
-    </collision>
-    <collision>
-      <origin rpy="0 0 0" xyz="0.05 -0.038 -0.06"/>
-      <geometry>
-        <sphere radius="0.005"/>
-      </geometry>
-    </collision>
-    <collision>
-      <origin rpy="0 0 0" xyz="0.112 0.027 -0.06"/>
-      <geometry>
-        <sphere radius="0.005"/>
-      </geometry>
-    </collision>
-    <collision>
-      <origin rpy="0 0 0" xyz="0.122 0.015 -0.05"/>
-      <geometry>
-        <sphere radius="0.005"/>
-      </geometry>
-    </collision>
-    <collision>
-      <origin rpy="0 0 0" xyz="0.125 0 -0.047"/>
-      <geometry>
-        <sphere radius="0.005"/>
-      </geometry>
-    </collision>
-    <collision>
-      <origin rpy="0 0 0" xyz="0.122 -0.015 -0.05"/>
-      <geometry>
-        <sphere radius="0.005"/>
-      </geometry>
-    </collision>
-    <collision>
-      <origin rpy="0 0 0" xyz="0.112 -0.027 -0.06"/>
-      <geometry>
-        <sphere radius="0.005"/>
-      </geometry>
-    </collision>
-    <inertial>
-      <origin xyz="3.460414800e-02 4.987565000e-06 -4.095111700e-02"/>
-      <mass value="6.616435000e-01"/>
-      <inertia ixx="4.316320200e-04" ixy="8.340871900e-08" ixz="4.556600800e-05" iyy="1.641839900e-03" iyz="-3.054166700e-08" izz="1.722959300e-03"/>
+    </collision>
+    <inertial>
+      <origin xyz="3.460414800e-02 4.987565000e-06 -4.095111700e-02" />
+      <mass value="6.616435000e-01" />
+      <inertia ixx="4.316320200e-04" ixy="8.340871900e-08" ixz="4.556600800e-05"
+                iyy="1.641839900e-03" iyz="-3.054166700e-08"
+                izz="1.722959300e-03" />
     </inertial>
   </link>
@@ -277,13 +236,15 @@
     </visual>
     <collision>
-      <origin rpy="1.5708 0 0" xyz="0 -0.05 -0.02"/>
-      <geometry>
-        <cylinder length="0.07" radius="0.04"/>
-      </geometry>
-    </collision>
-    <inertial>
-      <origin xyz="-1.141350800e-03 -7.948863700e-02 -2.579253000e-02"/>
-      <mass value="1.134347800e+00"/>
-      <inertia ixx="1.413427800e-03" ixy="-1.539744300e-05" ixz="-1.209053000e-05" iyy="1.011315000e-03" iyz="-1.526223400e-04" izz="1.066188000e-03"/>
+      <origin xyz="0 -0.05 -0.02" rpy="1.5708 0 0"/>
+      <geometry>
+        <cylinder radius="0.04" length="0.07"/>
+      </geometry>
+    </collision>
+    <inertial>
+       <origin xyz="-1.141350800e-03 -7.948863700e-02 -2.579253000e-02" />
+       <mass value="1.134347800e+00" />
+       <inertia ixx="1.413427800e-03" ixy="-1.539744300e-05" ixz="-1.209053000e-05"
+       iyy="1.011315000e-03" iyz="-1.526223400e-04"
+       izz="1.066188000e-03" />
     </inertial>
   </link>
@@ -304,7 +265,9 @@
     </visual>
     <inertial>
-      <origin xyz="1.451722900e-02 -2.959881100e-06 -7.908222600e-02"/>
-      <mass value="1.553530600e+00"/>
-      <inertia ixx="2.895595600e-03" ixy="2.404258600e-07" ixz="-7.419442800e-05" iyy="3.373592400e-03" iyz="2.679668900e-07" izz="1.929922100e-03"/>
+       <origin xyz="1.451722900e-02 -2.959881100e-06 -7.908222600e-02" />
+       <mass value="1.553530600e+00" />
+       <inertia ixx="2.895595600e-03" ixy="2.404258600e-07" ixz="-7.419442800e-05"
+       iyy="3.373592400e-03" iyz="2.679668900e-07"
+       izz="1.929922100e-03" />
     </inertial>
   </link>
@@ -325,13 +288,15 @@
     </visual>
     <collision>
-      <origin rpy="0 0 0" xyz="0.0 0 -0.08"/>
-      <geometry>
-        <cylinder length="0.13" radius="0.045"/>
-      </geometry>
-    </collision>
-    <inertial>
-      <origin xyz="-1.979799000e-03 4.937156100e-03 -1.811430100e-01"/>
-      <mass value="1.898213600e+00"/>
-      <inertia ixx="1.106355100e-02" ixy="6.007863900e-05" ixz="-4.880601900e-04" iyy="1.147669300e-02" iyz="6.113904800e-04" izz="1.632776900e-03"/>
+      <origin xyz="0.0 0 -0.08" rpy="0 0 0"/>
+      <geometry>
+        <cylinder radius="0.045" length="0.13"/>
+      </geometry>
+    </collision>
+    <inertial>
+       <origin xyz="-1.979799000e-03 4.937156100e-03 -1.811430100e-01" />
+       <mass value="1.898213600e+00" />
+       <inertia ixx="1.106355100e-02" ixy="6.007863900e-05" ixz="-4.880601900e-04"
+       iyy="1.147669300e-02" iyz="6.113904800e-04"
+       izz="1.632776900e-03" />
     </inertial>
   </link>
@@ -352,14 +317,16 @@
     </visual>
     <collision>
-      <origin rpy="0 0 0" xyz="0.0 0 -0.10"/>
-      <geometry>
-        <cylinder length="0.18" radius="0.04"/>
-      </geometry>
-    </collision>
-    <inertial>
-      <origin xyz="-3.870294200e-04 -3.148109200e-03 -1.238798000e-01"/>
-      <mass value="2.340311200e+00"/>
-      <inertia ixx="1.081088800e-02" ixy="-1.641625300e-04" ixz="-2.747466700e-04" iyy="1.105245000e-02" iyz="3.835456300e-04" izz="2.561741000e-03"/>
-    </inertial>
+      <origin xyz="0.0 0 -0.10" rpy="0 0 0"/>
+      <geometry>
+        <cylinder radius="0.04" length="0.18"/>
+      </geometry>
+    </collision>
+     <inertial>
+        <origin xyz="-3.870294200e-04 -3.148109200e-03 -1.238798000e-01" />
+        <mass value="2.340311200e+00" />
+        <inertia ixx="1.081088800e-02" ixy="-1.641625300e-04" ixz="-2.747466700e-04"
+        iyy="1.105245000e-02" iyz="3.835456300e-04"
+        izz="2.561741000e-03" />
+     </inertial>
   </link>
   <joint name="right_knee_joint" type="revolute">
@@ -385,7 +352,9 @@
     </collision>-->
     <inertial>
-      <origin xyz="5.032473200e-03 -3.766079000e-05 2.402319500e-03"/>
-      <mass value="6.779372600e-01"/>
-      <inertia ixx="3.704684500e-04" ixy="-1.179149700e-06" ixz="4.766622000e-05" iyy="4.135993600e-04" iyz="5.727227700e-07" izz="4.302869000e-04"/>
+      <origin xyz="5.032473200e-03 -3.766079000e-05 2.402319500e-03" />
+      <mass value="6.779372600e-01" />
+      <inertia ixx="3.704684500e-04" ixy="-1.179149700e-06" ixz="4.766622000e-05"
+                iyy="4.135993600e-04" iyz="5.727227700e-07"
+                izz="4.302869000e-04" />
     </inertial>
   </link>
@@ -405,68 +374,16 @@
       <material name="white"/>
     </visual>
-    <!-- <collision>
+    <collision>
       <origin rpy="0 0 0" xyz="0 0 0"/>
       <geometry>
         <mesh filename="package://ai_sapiens_description/meshes/k1_rev1/right_ankle_roll_link.stl" scale="0.001 0.001 0.001"/>
       </geometry>
-    </collision> -->
-    <collision>
-      <origin rpy="0 0 0" xyz="-0.047 0.025 -0.06"/>
-      <geometry>
-        <sphere radius="0.005"/>
-      </geometry>
-    </collision>
-    <collision>
-      <origin rpy="0 0 0" xyz="-0.047 -0.025 -0.06"/>
-      <geometry>
-        <sphere radius="0.005"/>
-      </geometry>
-    </collision>
-    <collision>
-      <origin rpy="0 0 0" xyz="0.05 0.038 -0.06"/>
-      <geometry>
-        <sphere radius="0.005"/>
-      </geometry>
-    </collision>
-    <collision>
-      <origin rpy="0 0 0" xyz="0.05 -0.038 -0.06"/>
-      <geometry>
-        <sphere radius="0.005"/>
-      </geometry>
-    </collision>
-    <collision>
-      <origin rpy="0 0 0" xyz="0.112 0.027 -0.06"/>
-      <geometry>
-        <sphere radius="0.005"/>
-      </geometry>
-    </collision>
-    <collision>
-      <origin rpy="0 0 0" xyz="0.122 0.015 -0.05"/>
-      <geometry>
-        <sphere radius="0.005"/>
-      </geometry>
-    </collision>
-    <collision>
-      <origin rpy="0 0 0" xyz="0.125 0 -0.047"/>
-      <geometry>
-        <sphere radius="0.005"/>
-      </geometry>
-    </collision>
-    <collision>
-      <origin rpy="0 0 0" xyz="0.122 -0.015 -0.05"/>
-      <geometry>
-        <sphere radius="0.005"/>
-      </geometry>
-    </collision>
-    <collision>
-      <origin rpy="0 0 0" xyz="0.112 -0.027 -0.06"/>
-      <geometry>
-        <sphere radius="0.005"/>
-      </geometry>
-    </collision>
-    <inertial>
-      <origin xyz="3.460414800e-02 4.987565000e-06 -4.095111700e-02"/>
-      <mass value="6.616435000e-01"/>
-      <inertia ixx="4.316320200e-04" ixy="8.340871900e-08" ixz="4.556600800e-05" iyy="1.641839900e-03" iyz="-3.054166700e-08" izz="1.722959300e-03"/>
+    </collision>
+    <inertial>
+      <origin xyz="3.460414800e-02 4.987565000e-06 -4.095111700e-02" />
+      <mass value="6.616435000e-01" />
+      <inertia ixx="4.316320200e-04" ixy="8.340871900e-08" ixz="4.556600800e-05"
+                iyy="1.641839900e-03" iyz="-3.054166700e-08"
+                izz="1.722959300e-03" />
     </inertial>
   </link>
@@ -506,7 +423,9 @@
     </collision>
     <inertial>
-      <origin xyz="-1.396563000e-02 6.013817200e-04 2.110737900e-01"/>
-      <mass value="7.719359000e+00"/>
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